Commit message: Added Hubo Head

File: model.urdf (robot description, URDF)
Before this commit: robot huboplus, 58 links, 57 joints
Links:
- removed link Body_HNR
Joints:
- removed joint HNR
- joint HNP: origin xyz=0 0 0 rpy=0 -0 0 -> xyz=0.0122581 0.0024526 0.196935 rpy=0 -0 0; parent Body_HNR -> Body_Torso
